File: KicadFiles/SingleBoardComputer/SingleBoardComputer.kicad_sch (KiCad schematic)
At the start: 86 parts, among them J1 USB_C_Receptacle_USB2.0_16P, J2 Conn_01x10_Pin, J3 Conn_01x06_Pin, SW1 SW_DPST_x2, U1 8468-11B1-RK-TP, U10 AS7C1026B-12JCN, U11 SST39SF040-70-4C-PHE, U12 SST39SF040-70-4C-PHE, U2 TPS630701RNMT, U3 FT240XS, U4 LD1117S33TR_SOT223, U5 8444-11B1-RK-TP, U6 4832-6000-CP, U7 4832-6000-CP, U8 MC68000FN, U9 XC9572XL-PC44, Y1 CXO_DIP8

Commit message: Schematic after corrections
Parts:
- removed D2, D3, D4, D5, D6: LED, LED_SMD:LED_0805_2012Metric_Pad1.15x1.40mm_HandSolder, symbol Device:LED
- removed R10, R11, R12, R13, R14: 1k, Resistor_SMD:R_0805_2012Metric_Pad1.20x1.40mm_HandSolder, symbol Device:R
- removed R15, R23, R24, R34, R35, R36, R37: 5.1k, Resistor_SMD:R_0805_2012Metric_Pad1.20x1.40mm_HandSolder, symbol Device:R
- added D? (x5): LED, LED_SMD:LED_0805_2012Metric_Pad1.15x1.40mm_HandSolder, symbol Device:LED
- added J? (x2): Conn_01x06_Pin, symbol Connector:Conn_01x06_Pin
- added R? (x5): 1k, Resistor_SMD:R_0805_2012Metric_Pad1.20x1.40mm_HandSolder, symbol Device:R
- added R?: 5.1k, Resistor_SMD:R_0805_2012Metric_Pad1.20x1.40mm_HandSolder, symbol Device:R
- added U?: TLV809EA46DBZR, Package_TO_SOT_SMD:SOT-23, symbol CustomComponents:TLV809EA46DBZR
- FB1: value FerriteBead -> MI0805K601R-10
Connections:
- net +3V3: now also R?.1
- net +5V: now also R9.1, R?.1; no longer D1.2 (A)
- net +5VD: now also R?.1
- net A1: now also J?.6 (Pin_6)
- net A19: no longer U11.1 (A18), U12.1 (A18)
- net A2: now also J?.5 (Pin_5)
- net A20: no longer U9.11 (P11)
- net A21: no longer U9.12 (P12)
- net A22: no longer U9.13 (P13)
- net A23: no longer U9.14 (P14)
- net A3: now also J?.4 (Pin_4)
- net A4: now also J?.3 (Pin_3)
- net A5: now also J?.2 (Pin_2)
- net A6: now also J?.1 (Pin_1)
- net CLK: now also U9.6 (I/O/GCK2), R?.1; no longer U9.7 (I/O/GCK3)
- net CPU_AS: now also U9.11 (P11); no longer U9.5 (I/O/GCK1)
- net CPU_DTACK: now also R28.2, U9.9 (P9); no longer R25.2, U9.4 (P4)
- net CPU_FC0: now also U9.22 (P22); no longer R31.2, U9.20 (P20)
- net CPU_FC1: no longer R32.2
- net CPU_FC2: now also U9.20 (P20); no longer R33.2, U9.22 (P22)
- net CPU_HALT: now also R32.2, U9.18 (P18), R?.1; no longer R30.2, U9.19 (P19)
- net CPU_IPL0: now also R31.2, U9.14 (P14); no longer R28.2, U9.1 (P1)
- net CPU_IPL1: now also R30.2, U9.13 (P13); no longer R27.2, U9.2 (P2)
- net CPU_IPL2: now also R29.2, U9.12 (P12); no longer R26.2, U9.3 (P3)
- net CPU_LDS: now also U9.1 (P1)
- net CPU_RST: now also R33.2, U9.19 (P19), R?.1; no longer R29.2, U9.18 (P18)
- net CPU_R/W: now also U9.37 (P37); no longer U9.6 (I/O/GCK2)
- net CPU_UDS: now also U9.2 (P2)
- net C_EN: now also R?.2
- net D0: now also R27.2, U9.39 (I/O/GSR), J?.6 (Pin_6)
- net D1: now also J?.5 (Pin_5)
- net D2: now also J?.4 (Pin_4)
- net D3: now also J?.3 (Pin_3)
- net D4: now also J?.2 (Pin_2)
- net D5: now also J?.1 (Pin_1)
- net GND: now also D1.1 (K), U11.1 (A18), U12.1 (A18), D?.1 (K), D?.1 (K), D?.1 (K), D?.1 (K), D?.1 (K), U?.1 (GND); no longer R9.2
- net RAM_CE: now also U9.5 (I/O/GCK1); no longer U9.25 (P25)
- net RAM_OE: now also U9.3 (P3); no longer U9.27 (P27)
- net RAM_WE: now also U9.4 (P4); no longer U9.26 (P26)
- net ROM_0_CE: now also R25.2, U9.44 (P44); no longer U9.28 (P28)
- net ROM_0_OE: now also R20.2, U9.42 (I/O/GTS1); no longer U9.33 (P33)
- net ROM_1_CE: now also R19.2, U9.43 (P43); no longer U9.29 (P29)
- net ROM_1_OE: now also R26.2, U9.40 (I/O/GTS2); no longer U9.34 (P34)
- net R_BTN: now also U9.7 (I/O/GCK3), U?.2 (~{Reset}); no longer R6.2, SW1.1 (A), U9.39 (I/O/GSR)
- net UTP_3V3: no longer U3.16 (~{RESET})
- net UTP_CBUS5: now also U9.33 (P33); no longer R19.2, U9.44 (P44)
- net UTP_CBUS6: now also U9.34 (P34); no longer R20.2, U9.43 (P43)
- net UTP_RD: now also U9.28 (P28); no longer U9.36 (P36)
- net UTP_RXF: now also U9.36 (P36); no longer U9.38 (P38)
- net UTP_SIWU: now also U9.38 (P38); no longer U9.9 (P9)
- net UTP_TXE: now also U9.35 (P35); no longer U9.37 (P37)
- net UTP_WR: now also U9.27 (P27); no longer U9.35 (P35)
- new net: D?.2 (A), R?.2 (x5)
- new net: D1.2 (A), R9.2
- new net: R6.2, SW1.1 (A), U?.3 (VDD)
- new net UTP_RST: U3.16 (~{RESET}), U9.29 (P29)
- no-connect marks 8 -> 6
Other:
- note added: "ABUS/DBUS Test Headers"
- moved on the sheet: C19, C20, C21, C22, D1, FB1, R16, R17, R18, R19, R20, R25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

Commit message: Correction Corrections
Parts:
- removed SW1: SW_DPST_x2, Button_Switch_SMD:SW_SPST_PTS647_Sx38, symbol Switch:SW_DPST_x2
- added SW1: SW_DPST_x2_Custom, Button_Switch_SMD:SW_SPST_PTS647_Sx38, symbol CustomComponents:SW_DPST_x2_Custom
- J4, J5: renamed from J?; footprint (none) -> Connector_PinHeader_2.54mm:PinHeader_1x06_P2.54mm_Vertical
- U3: renamed from U2; footprint RNM0015A -> CustomComponents:RNM0015A
- U6: renamed from U5; footprint Package_LCC:PLCC-44_THT-Socket -> TO_11B1-RK-TP_3MM
- gave numbers to parts that had none: 12
- renumbered C23 to C20, C24 to C21, C20 to C22, C21 to C23, C22 to C24, R29 to R15, R30 to R16, R31 to R17, R32 to R18, R33 to R19, R25 to R21, R19 to R22, R20 to R23, R26 to R24, R27 to R25, R28 to R26, R16 to R27, R17 to R28, R18 to R29, U9 to U11, U11 to U12, U12 to U13, U3 to U4, U4 to U5, U6 to U7, U7 to U8, U8 to U9
Connections:
- net A19: now also U11.25 (P25)
- net A20: now also U11.26 (P26)
- net GND: now also SW1.2 (B)
- net at R6.2, U2.3 (VDD): now also SW1.1 (A)
- net A21: no longer names the net of U9.53 (A21)
- net A22: no longer names the net of U9.54 (A22)
- net A23: no longer names the net of U9.55 (A23)
- no-connect marks 6 -> 181
Other:
- moved on the sheet: U8

Commit message: PCB done
Changed lines of the file:
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@@
 			)
 		)
-		(property "Datasheet" "~"
+		(property "Datasheet" "https://www.digikey.com/en/products/detail/amphenol-cs-commercial-products/G800W302018EU/17069165"
 			(at 262.89 151.13 0)
 			(effects
@@
 			)
 		)
-		(property "Datasheet" "https://www.digikey.com/en/products/detail/adam-tech/PH1-10-UA/9830653?s=N4IgjCBcoGwJxVAYygMwIYBsDOBTANCAPZQDaIALGGABxwDsIAuoQA4AuUIAyuwE4BLAHYBzEAF9CNGohApIGHAWJkQMAMxwaMZm06Qe-YWMkg4ABlnzFeQiUjlNMGAFZdIDl16DREwmHh1KzQsWxUHEHUwODgAJgQWD31DHxN-egtghVDle3IGWJ1EzwNvYz9wLQRoORClO1VLJlNY81iIGuschoiqehoXBL0vI19TAFoZTrqwvJBWl0ZmwnGdach%2BAFdc1SDlkHHYrK2diLd98erkKBOe8ghm8XEgA"
+		(property "Datasheet" "https://www.digikey.com/en/products/detail/amphenol-cs-fci/10129378-910002BLF/7915958"
 			(at 180.34 105.41 0)
 			(effects
@@
 			)
 		)
-		(property "Datasheet" "https://www.digikey.com/en/products/detail/adam-tech/ADT-AMP1251106S4BS165A1/9832042"
+		(property "Datasheet" "https://www.digikey.com/en/products/detail/amphenol-cs-commercial-products/G800W302018EU/17069165"
 			(at 290.83 109.22 0)
 			(effects
@@
 		(lib_id "Device:R")
 		(at 208.28 191.77 0)
+		(mirror y)
 		(unit 1)
 		(exclude_from_sim no)
@@
 		(dnp yes)
 		(property "Reference" "R20"
-			(at 208.026 195.326 0)
+			(at 208.534 195.326 0)
 			(effects
 				(font
@@
 		)
 		(property "Footprint" "Resistor_SMD:R_0805_2012Metric_Pad1.20x1.40mm_HandSolder"
-			(at 206.502 191.77 90)
+			(at 210.058 191.77 90)
 			(effects
 				(font
@@
 			)
 		)
-		(property "Datasheet" "TPS630701RNMT"
+		(property "Datasheet" "https://www.digikey.com/en/products/detail/texas-instruments/TPS630701RNMT/6193742"
 			(at 148.59 48.26 0)
 			(effects
@@
 			)
 		)
-		(property "Datasheet" "~"
+		(property "Datasheet" "https://www.digikey.com/en/products/detail/amphenol-cs-commercial-products/G800W302018EU/17069165"
 			(at 224.79 151.13 0)
 			(effects
