File: KicadFiles/SingleBoardComputer/SingleBoardComputer.kicad_sch (KiCad schematic)
At the start: 83 parts, among them J1 USB_C_Receptacle_USB2.0_16P, J2 Conn_01x10_Pin, J3 Conn_01x06_Pin, J4 Conn_01x06_Pin, J5 Conn_01x06_Pin, SW1 SW_DPST_x2_Custom, U1 8468-11B1-RK-TP, U10 AS7C1026B-12JCN, U11 XC9572XL-PC44, U12 SST39SF040-70-4C-PHE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

Commit message: Purchase 1
Parts:
- C11: LCSC PN (none) -> C155422
- L1: LCSC PN (none) -> C3033018
- U3: LCSC PN (none) -> C181473
- U4: LCSC PN (none) -> C69082
- U5: LCSC PN (none) -> LD1117S33TR
