File: KicadFiles/SingleBoardComputer/SingleBoardComputer.kicad_pcb (KiCad board)
At the start: 2 copper layers, 95 x 95 mm, 97 parts, among them J1 USB_C_Receptacle_USB2.0_16P, J2 Conn_01x10_Pin, J3 Conn_01x06_Pin, J4 Conn_01x06_Pin, J5 Conn_01x06_Pin, SW1 SW_DPST_x2, SW1 SW_DPST_x2_Custom, U10 AS7C1026B-12JCN, U11 XC9572XL-PC44, U12 SST39SF040-70-4C-PHE, U13 SST39SF040-70-4C-PHE, U2 TLV809EA46DBZR, U3 TPS630701RNMT, U4 FT240XS, U5 LD1117S33TR_SOT223, U9 MC68000FN, Y1 CXO_DIP8

Commit message: PCB done
Parts:
- removed the D2 at (78.2, 79.3)
- removed the D2 at (111.2, 63.9)
- removed the D3 at (166.0, 47.9)
- removed the D3 at (78.2, 82.4)
- removed the D4 at (78.2, 85.4)
- removed the D4 at (194.3, 75.5)
- removed the D5 at (168.2, 62.6)
- removed the D5 at (78.2, 88.5)
- removed the D6 at (78.2, 91.5)
- removed the D6 at (171.7, 62.6)
- removed the R10 at (73.4, 79.3)
- removed the R10 at (115.5, 62.3)
- removed the R11 at (73.4, 82.2)
- removed the R11 at (166.0, 53.0)
- removed the R12 at (73.4, 85.2)
- removed the R12 at (194.3, 70.9)
- removed the R13 at (168.2, 67.2)
- removed the R13 at (73.4, 88.1)
- removed the R14 at (73.4, 91.1)
- removed the R14 at (171.6, 67.2)
- removed the R15 at (182.3, 63.8)
- removed the R15 at (210.1, 78.5)
- removed the R23 at (136.9, 61.5)
- removed the R24 at (220.3, 78.5)
- removed the R24 at (137.1, 66.2)
- removed R34, R35, R36, R37: 5.1k, Resistor_SMD:R_0805_2012Metric_Pad1.20x1.40mm_HandSolder
- removed the SW1 at (181.6, 59.5)
- removed the SW1 at (3.67, 2.73)
- added D2: LED, LED_SMD:LED_0805_2012Metric_Pad1.15x1.40mm_HandSolder, F.Cu at (105.6, 67.4)
- added D3: LED, LED_SMD:LED_0805_2012Metric_Pad1.15x1.40mm_HandSolder, F.Cu at (165.6, 51.0)
- added D4: LED, LED_SMD:LED_0805_2012Metric_Pad1.15x1.40mm_HandSolder, F.Cu at (194.1, 66.2)
- added D5: LED, LED_SMD:LED_0805_2012Metric_Pad1.15x1.40mm_HandSolder, F.Cu at (173.4, 75.6)
- added D6: LED, LED_SMD:LED_0805_2012Metric_Pad1.15x1.40mm_HandSolder, F.Cu at (176.6, 75.7)
- added R10: 1k, Resistor_SMD:R_0805_2012Metric_Pad1.20x1.40mm_HandSolder, F.Cu at (105.5, 64.1)
- added R11: 1k, Resistor_SMD:R_0805_2012Metric_Pad1.20x1.40mm_HandSolder, F.Cu at (165.7, 56.3)
- added R12: 1k, Resistor_SMD:R_0805_2012Metric_Pad1.20x1.40mm_HandSolder, F.Cu at (194.2, 71.4)
- added R13: 1k, Resistor_SMD:R_0805_2012Metric_Pad1.20x1.40mm_HandSolder, F.Cu at (173.4, 70.7)
- added R14: 1k, Resistor_SMD:R_0805_2012Metric_Pad1.20x1.40mm_HandSolder, F.Cu at (176.3, 70.7)
- added R15: 5.1k, Resistor_SMD:R_0805_2012Metric_Pad1.20x1.40mm_HandSolder, F.Cu at (163.0, 76.8)
- added R24: 5.1k, Resistor_SMD:R_0805_2012Metric_Pad1.20x1.40mm_HandSolder, F.Cu at (153.4, 92.8)
- added SW1: SW_DPST_x2_Custom, Button_Switch_SMD:SW_SPST_PTS647_Sx38, F.Cu at (178.9, 61.1)
- moved J5 137.9 mm to (194.4, 88.7), turned to 180 degrees
- moved R20 116.0 mm to (185.3, 63.8), turned to 180 degrees
- moved U2 91.8 mm to (172.9, 62.0), turned to -90 degrees
- moved J4 81.8 mm to (127.7, 120.5), turned to 180 degrees
- moved R25 63.2 mm to (157.0, 106.7), turned to 90 degrees
- moved R26 46.9 mm to (170.3, 83.2)
- moved R16 46.6 mm to (160.2, 76.5), turned to 90 degrees
- moved R23 43.6 mm to (123.4, 92.8), turned to -90 degrees
- moved R18 41.8 mm to (172.6, 66.6), turned to 180 degrees
- moved R17 40.7 mm to (163.9, 84.6), turned to -90 degrees
- moved R22 40.3 mm to (150.2, 92.8), turned to -90 degrees
- moved R21 38.8 mm to (119.7, 92.8), turned to -90 degrees
- moved R6 38.6 mm to (168.9, 61.4)
- moved R19 35.7 mm to (176.5, 66.6), turned to 180 degrees
- moved C15 12.7 mm to (194.9, 109.5), turned to -90 degrees
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Routing:
- net +5V: track 303.5 -> 726.8 mm, vias 6 -> 17
- net GND: track 39.8 -> 338.1 mm, vias 2 -> 98
- net CPU_IPL2: track 128.8 -> 66.0 mm, vias 2 -> 3
- net +3V3: track 45.9 -> 103.7 mm, vias 1 -> 3
- net CPU_IPL0: track 127.7 -> 76.1 mm
- net CLK: track 71.3 -> 122.0 mm, vias 2 -> 3
- net CPU_IPL1: track 118.1 -> 69.6 mm, vias 1 -> 0
- net D1: track 105.7 -> 143.1 mm
- net A20: track 67.9 -> 97.6 mm
- net D2: track 102.2 -> 131.9 mm
- net CPU_HALT: track 64.6 -> 93.9 mm, vias 2 -> 5
- net ROM_0_CE: track 96.2 -> 67.6 mm, vias 4 -> 3
- net ROM_0_OE: track 100.0 -> 72.2 mm, vias 11 -> 3
- net CPU_LDS: track 64.5 -> 90.2 mm
- net Net-(J1-SHIELD): track 2.93 -> 27.3 mm, vias 0 -> 3
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Other:
- board text added: "AS"
- board text added: "CBUS5"
- board text added: "CBUS6"
- board text added: "CLK"
- board text added: "CPLD"
- board text added: "CPU"
- board text added: "C_EN"
- board text added: "D0"
- board text added: "D1"
- board text added: "D2"
- board text added: "D3"
- board text added: "D4"
- board text added: "D5"
- board text added: "DTACK"
- board text added: "GND"
- board text added: "HALT"
- board text added: "IPL0"
- board text added: "IPL1"
- board text added: "IPL2"
- board text added: "R/W"
- board text added: "RAM"
- board text added: "RD"
- board text added: "ROM LOWER"
- board text added: "ROM UPPER"
- board text added: "ROM_0_CE"
- board text added: "ROM_0_OE"
- board text added: "ROM_1_CE"
- board text added: "ROM_1_OE"
- board text added: "RST"
- board text added: "RXF"
- board text added: "SAMUEL ARMSTRONG LETU SP 2025 Single Board Computer Rev 2"
- board text added: "TCK"
- board text added: "TDI"
- board text added: "TDO"
- board text added: "TMS"
- board text added: "TXE"
- board text added: "USB"
- board text added: "USB To Parallel"
- board text added: "VCC"
- board text added: "WR"

Commit message: Purchase 1
Parts:
- moved R16 0.23 mm to (160.0, 76.7)
- moved R15 0.21 mm to (162.9, 76.6)
- moved R3 0.17 mm to (111.9, 47.1)
- moved R13 0.15 mm to (173.5, 70.5)
- moved R14 0.11 mm to (176.3, 70.6)
Routing:
- net GND: track 338.1 -> 345.9 mm, vias 98 -> 101
- net +5V: track 726.8 -> 731.9 mm
- net +3V3: track 103.7 -> 105.6 mm
- net CPU_UDS: track 78.3 -> 79.6 mm
- net CPU_FC2: track 87.6 -> 88.9 mm
- net CLK: track 122.0 -> 120.7 mm
- net D6: track 130.0 -> 131.2 mm
- net D7: track 138.8 -> 140.0 mm
- net ROM_0_OE: track 72.2 -> 71.1 mm
- net D4: track 138.8 -> 139.8 mm
- net D3: track 143.9 -> 144.8 mm
- net CPU_RST: track 92.0 -> 91.0 mm
- net D15: track 119.5 -> 118.6 mm
- net CPU_DTACK: track 82.0 -> 82.8 mm
- net RAM_OE: track 33.9 -> 33.0 mm
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